File: .review_backup_20260616/MCU_Core.kicad_sch (KiCad schematic)
At the start: 30 parts, among them J33 Dev/SWD header, U2 W25Q16JVUXIQ, U3 RP2040, Y1 ABM8-272-T3

Commit message: checking
Parts:
- C1, C17: value 1u -> 10u
Connections:
- net +3V3: no longer C1.1, C17.1
- net GND: no longer C17.2
- net USB_DM: no longer R4.1
- net USB_DP: no longer R3.1
