File: .review_backup_20260616/defcon_badge.kicad_pcb (KiCad board)
At the start: 4 copper layers, 88 x 54 mm, 81 parts, among them J10 USB_C_Receptacle_GCT_USB4085, J11 JST-PH 2P, J20 AMPHENOL_10038075-D0P, J30 SAO 2x3, J31 microSD, SW1 SS-12D00, SW20 TS-1187A, SW21 TS-1187A, SW22 TS-1187A, SW23 TS-1187A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

Commit message: checking
Parts:
- C1, C17: value 1u -> 10u
- moved C3 9.92 mm to (133.1, 106.0)
- moved C2 8.34 mm to (137.7, 104.4), turned to 180 degrees
- moved Y1 7.77 mm to (135.8, 106.9), turned to 180 degrees
- moved R5 7.07 mm to (133.2, 104.3), turned to 180 degrees
Connections:
- net /MCU_Core/BOOTSEL renamed BOOTSEL
- C1 pad 1: +3V3 -> unconnected-(C1-Pad1)
- C17 pad 1: +3V3 -> unconnected-(C17-Pad1)
- C17 pad 2: GND -> unconnected-(C17-Pad2)
- J10 pad A5: /Power/CC1 -> /Power/CC2
- J10 pad A6: /MCU_Core/USB_DP -> Net-(U3-USB_DP)
- J10 pad A7: /MCU_Core/USB_DM -> Net-(U3-USB_DM)
- J10 pad A8: unconnected-(J10-SBU1-PadA8) -> (no net)
- J10 pad B6: /MCU_Core/USB_DP -> Net-(U3-USB_DP)
- J10 pad B7: /MCU_Core/USB_DM -> Net-(U3-USB_DM)
- J10 pad B8: unconnected-(J10-SBU2-PadB8) -> (no net)
- R10 pad 1: /Power/CC1 -> GND
- R3 pad 1: /MCU_Core/USB_DP -> unconnected-(R3-Pad1)
- R4 pad 1: /MCU_Core/USB_DM -> unconnected-(R4-Pad1)
- U10 pad 8: /Power/VBUS -> /Power/+3V3
- U3 pad 30: /IO/BTN_SYNC -> /MCU_Core/GPIO19
