File: defcon_badge/IO.kicad_sch (KiCad schematic)
At the start: 8 parts, among them J30 SAO 2x3, J31 microSD, J32 UART debug, SW20 TS-1187A, SW21 TS-1187A, SW22 TS-1187A

Commit message: checking
Parts:
- added SW23: TS-1187A, Button_Switch_SMD:SW_SPST_TL3342, symbol Switch:SW_Push
Connections:
- net GND: now also SW23.2
- new net BTN_SYNC: SW23.1
Changed lines of the file:
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@@
+	)
+	(symbol
+		(lib_id "Switch:SW_Push")
+		(at 110.49 59.69 0)
+		(unit 1)
+		(body_style 1)
+		(exclude_from_sim no)
+		(in_bom yes)
+		(on_board yes)
+		(in_pos_files yes)
+		(dnp no)
+		(fields_autoplaced yes)
+		(property "Reference" "SW23" (at 110.49 52.07 0) (effects (font (size 1.27 1.27))))
+		(property "Value" "TS-1187A" (at 110.49 67.31 0) (effects (font (size 1.27 1.27))))
+		(property "Footprint" "Button_Switch_SMD:SW_SPST_TL3342" (at 110.49 59.69 0) (show_name no) (hide yes) (effects (font (size 1.27 1.27))))
+		(property "Datasheet" "" (at 110.49 59.69 0) (show_name no) (hide yes) (effects (font (size 1.27 1.27))))
+		(property "Description" "Sync button (SYNC), 6mm tactile" (at 110.49 59.69 0) (show_name no) (hide yes) (effects (font (size 1.27 1.27))))
+		(property "MPN" "TS-1187A-B-A-B" (at 110.49 59.69 0) (show_name no) (hide yes) (effects (font (size 1.27 1.27))))
+		(property "LCSC" "C455257" (at 110.49 59.69 0) (show_name no) (hide yes) (effects (font (size 1.27 1.27))))
+		(pin "1")
+		(pin "2")
+		(instances
+			(project "defcon_badge"
+				(path "/8c0b3d8b-46d3-4173-ab1e-a61765f77d61/608539de-722a-4bca-b1da-2c313b60cd6f"
+					(reference "SW23")
+					(unit 1)
+				)
+			)
+		)
 	)
 	(symbol
@@
 				(path "/8c0b3d8b-46d3-4173-ab1e-a61765f77d61/608539de-722a-4bca-b1da-2c313b60cd6f"
 					(reference "#PWR_SW22")
+					(unit 1)
+				)
+			)
+		)
+	)
+	(symbol
+		(lib_id "power:GND")
+		(at 118.11 59.69 0)
+		(unit 1)
+		(body_style 1)
+		(exclude_from_sim no)
+		(in_bom yes)
+		(on_board yes)
+		(in_pos_files yes)
+		(dnp no)
+		(fields_autoplaced yes)
+		(property "Reference" "#PWR_SW23" (at 118.11 52.07 0) (effects (font (size 1.27 1.27))))
+		(property "Value" "GND" (at 118.11 67.31 0) (effects (font (size 1.27 1.27)) (hide yes)))
+		(property "Footprint" "" (at 118.11 59.69 0) (show_name no) (hide yes) (effects (font (size 1.27 1.27))))
+		(property "Datasheet" "" (at 118.11 59.69 0) (show_name no) (hide yes) (effects (font (size 1.27 1.27))))
+		(property "Description" "" (at 118.11 59.69 0) (show_name no) (hide yes) (effects (font (size 1.27 1.27))))
+		(pin "1")
+		(instances
+			(project "defcon_badge"
+				(path "/8c0b3d8b-46d3-4173-ab1e-a61765f77d61/608539de-722a-4bca-b1da-2c313b60cd6f"
+					(reference "#PWR_SW23")
 					(unit 1)
 				)
@@
 	(wire (pts (xy 85.09 59.69) (xy 82.55 59.69)) (stroke (width 0) (type default)))
 	(wire (pts (xy 95.25 59.69) (xy 97.79 59.69)) (stroke (width 0) (type default)))
+	(wire (pts (xy 105.41 59.69) (xy 102.87 59.69)) (stroke (width 0) (type default)))
+	(wire (pts (xy 115.57 59.69) (xy 118.11 59.69)) (stroke (width 0) (type default)))
 	(wire (pts (xy 124.46 67.31) (xy 121.92 67.31)) (stroke (width 0) (type default)))
 	(wire (pts (xy 137.16 67.31) (xy 139.70 67.31)) (stroke (width 0) (type default)))
@@
 	(wire (pts (xy 35.56 110.49) (xy 38.10 110.49)) (stroke (width 0) (type default)))
 	(wire (pts (xy 35.56 119.38) (xy 38.10 119.38)) (stroke (width 0) (type default)))
+	(wire (pts (xy 35.56 127.00) (xy 38.10 127.00)) (stroke (width 0) (type default)))
 	(wire (pts (xy 35.56 134.62) (xy 38.10 134.62)) (stroke (width 0) (type default)))
 	(wire (pts (xy 35.56 144.78) (xy 38.10 144.78)) (stroke (width 0) (type default)))
@@
 	(label "BTN_VOL_UP" (at 62.23 59.69 0) (effects (font (size 1.27 1.27)) (justify left bottom)))
 	(label "BTN_VOL_DN" (at 82.55 59.69 0) (effects (font (size 1.27 1.27)) (justify left bottom)))
+	(label "BTN_SYNC" (at 102.87 59.69 0) (effects (font (size 1.27 1.27)) (justify left bottom)))
 	(label "+3V3" (at 139.70 67.31 0) (effects (font (size 1.27 1.27)) (justify left bottom)))
 	(label "SAO_SDA" (at 121.92 69.85 0) (effects (font (size 1.27 1.27)) (justify left bottom)))
@@
 	(label "BTN_VOL_UP" (at 38.10 110.49 0) (effects (font (size 1.27 1.27)) (justify left bottom)))
 	(label "BTN_VOL_DN" (at 38.10 119.38 0) (effects (font (size 1.27 1.27)) (justify left bottom)))
+	(label "BTN_SYNC" (at 38.10 127.00 0) (effects (font (size 1.27 1.27)) (justify left bottom)))
 	(label "SAO_SDA" (at 38.10 134.62 0) (effects (font (size 1.27 1.27)) (justify left bottom)))
 	(label "SAO_SCL" (at 38.10 144.78 0) (effects (font (size 1.27 1.27)) (justify left bottom)))
@@
 	(hierarchical_label "BTN_VOL_UP" (shape output) (at 35.56 110.49 0) (effects (font (size 1.524 1.524)) (justify left)))
 	(hierarchical_label "BTN_VOL_DN" (shape output) (at 35.56 119.38 0) (effects (font (size 1.524 1.524)) (justify left)))
+	(hierarchical_label "BTN_SYNC" (shape output) (at 35.56 127.00 0) (effects (font (size 1.524 1.524)) (justify left)))
 	(hierarchical_label "SAO_SDA" (shape bidirectional) (at 35.56 134.62 0) (effects (font (size 1.524 1.524)) (justify left)))
 	(hierarchical_label "SAO_SCL" (shape input) (at 35.56 144.78 0) (effects (font (size 1.524 1.524)) (justify left)))
