File: defcon_badge/Power.kicad_sch (KiCad schematic)
At the start: 15 parts, among them J10 USB_C_Receptacle_USB2.0_16P, J11 JST-PH 2P, SW1 SS-12D00, U10 TP4056, U11 ME6211C33M5G

Commit message: checking
Connections:
- net +3V3: no longer U10.8 (CE)
- net GND: no longer J10.A5 (CC1), R10.1
- net VBUS: now also U10.8 (CE)
- new net CC1: J10.A5 (CC1), R10.1
