File: defcon_badge/defcon_badge.kicad_sch (KiCad schematic)
At the start: 0 parts

Commit message: checking
Other:
- sheet IO ports: added BTN_SYNC; removed none
- sheet MCU_Core ports: added BTN_SYNC; removed none
Changed lines of the file:
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@@
+	(wire
+		(pts
+			(xy 150.5 236.22) (xy 165.1 236.22)
+		)
+		(stroke
+			(width 0)
+			(type default)
+		)
+	)
 	(wire
 		(pts
@@
 			)
 		)
+		(pin "BTN_SYNC" output
+			(at 150.5 236.22 0)
+			(effects
+				(font
+					(size 1.27 1.27)
+				)
+				(justify right)
+			)
+		)
 	)
 	(sheet
@@
 			(effects
 				(font
+					(size 1.27 1.27)
+				)
+				(justify left)
+			)
+		)
+		(pin "BTN_SYNC" input
+			(at 165.1 236.22 180)
+			(effects
+				(font
