File: defcon_badge/Audio.kicad_sch (KiCad schematic)
At the start: 16 parts, among them J5 SJ1-3523N, U5 TM8211, U6 TDA1308

Commit message: hardware: rev-2 bring-up updates, fab outputs, and the QR assets
Schematic/PCB updates accumulated during rev-2 bring-up and routing, plus
the rev-2 fabrication outputs (gerbers, placement) and the QR code that is
silkscreened on the board and points at this repository.

Repo hygiene for that audience: session-log text files removed from the
root, .DS_Store and the extracted fab directory ignored, fab zip rebuilt
without __MACOSX cruft.

Co-Authored-By: Claude Fable 5 <noreply@anthropic.com>
Parts:
- U6: footprint Package_SO:SOIC-8_3.9x4.9mm_P1.27mm -> Package_SO:TSSOP-8_3x3mm_P0.65mm
Changed lines of the file:
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@@
 			)
 		)
-		(property "Footprint" "Package_SO:SOIC-8_3.9x4.9mm_P1.27mm"
+		(property "Footprint" "Package_SO:TSSOP-8_3x3mm_P0.65mm"
 			(at 144.78 80.01 0)
 			(hide yes)
@@
 			)
 		)
-		(pin "R2"
-		)
-		(pin "D"
-		)
 		(pin "T"
