File: defcon_badge/MCU_Core.kicad_sch (KiCad schematic)
At the start: 30 parts, among them U2 W25Q16JVUXIQ, U3 RP2040, Y1 ABM8-272-T3

Commit message: Routing redo
Parts:
- removed C17: 1u, Capacitor_SMD:C_0805_2012Metric, symbol Device:C
- removed C4: 10u, Capacitor_SMD:C_0805_2012Metric, symbol Device:C
- renumbered C6 to C10, C7 to C11, C8 to C12, C9 to C13, C10 to C14, C11 to C15, C12 to C16, C14 to C17, C16 to C18, C2 to C5, C3 to C6, C1 to C7, C5 to C9, R1 to R10, R2 to R11, R5 to R12, R3 to R13, R4 to R14, R6 to R15, U2 to U3, U3 to U4
Connections:
- net GPIO25 is gone; now on net BTN_CH: U4.18 (GPIO15)
- net BTN_CH: no longer U4.15 (GPIO12)
- net BTN_SYNC: now also U4.15 (GPIO12); no longer U4.30 (GPIO19)
- net BTN_VOL_DN: now also U4.16 (GPIO13); no longer U4.17 (GPIO14)
- net BTN_VOL_UP: now also U4.17 (GPIO14); no longer U4.16 (GPIO13)
- new net GPIO19: U4.30 (GPIO19)
