File: defcon_badge/MCU_Core.kicad_sch (KiCad schematic)
At the start: 28 parts, among them U3 W25Q16JVUXIQ, U4 RP2040, Y1 ABM8-272-T3

Commit message: hardware: rev-2 bring-up updates, fab outputs, and the QR assets
Schematic/PCB updates accumulated during rev-2 bring-up and routing, plus
the rev-2 fabrication outputs (gerbers, placement) and the QR code that is
silkscreened on the board and points at this repository.

Repo hygiene for that audience: session-log text files removed from the
root, .DS_Store and the extracted fab directory ignored, fab zip rebuilt
without __MACOSX cruft.

Co-Authored-By: Claude Fable 5 <noreply@anthropic.com>
Parts:
- added C8: 100nF, Capacitor_SMD:C_0402_1005Metric, symbol Device:C
- added R23, R8, R9: 10k, Resistor_SMD:R_0402_1005Metric, symbol Device:R
- TP1, TP2: footprint TestPoint_Pad_D1.5mm -> TestPoint:TestPoint_Pad_D1.5mm
- U3: value W25Q16JVUXIQ -> WM2606220057; footprint Package_SON:Winbond_USON-8-1EP_3x2mm_P0.5mm_EP0.2x1.6mm -> Package_SO:SOIC-8_5.3x5.3mm_P1.27mm
Connections:
- net GND: now also C8.2
- net RUN: now also C8.1
- net SD_CS: now also R8.2
- net SD_MISO: now also R9.2
- net SD_MOSI: now also R23.2
- new net +3.3V: R23.1, R8.1, R9.1
