File: RP2040_minimal_r2.kicad_sch (KiCad schematic)
At the start: 34 parts, among them J1 USB_B_Micro, J2 Conn_01x02, J3 Conn_02x18_Odd_Even, J4 Conn_02x18_Odd_Even, U1 NCP1117-3.3_SOT223, U2 W25Q128JVS, U3 RP2040, Y1 ABM8-272-T3

Commit message: hardware: rev-2 bring-up updates, fab outputs, and the QR assets
Schematic/PCB updates accumulated during rev-2 bring-up and routing, plus
the rev-2 fabrication outputs (gerbers, placement) and the QR code that is
silkscreened on the board and points at this repository.

Repo hygiene for that audience: session-log text files removed from the
root, .DS_Store and the extracted fab directory ignored, fab zip rebuilt
without __MACOSX cruft.

Co-Authored-By: Claude Fable 5 <noreply@anthropic.com>
Parts:
- U2: value W25Q128JVS -> WM2606220057; footprint Package_SO:SOIC-8_5.23x5.23mm_P1.27mm -> Package_SO:SOIC-8_5.3x5.3mm_P1.27mm
